File: mini-pcie-breakout.kicad_sch (KiCad schematic)
At the start: 28 parts, among them J1 miniPCIe, J2 RX, J3 TX, J4 CLK, U1 AMS1117-1.5

Commit message: Add half-size mini PCIe support
Parts:
- added H11, H12: M3, MountingHole:MountingHole_3.2mm_M3, symbol Mechanical:MountingHole
